Commit message: orientacio robot

File: src/rubot_mecanum_description/urdf/rubot.urdf (robot description, URDF)
Before this commit: robot nexus, 8 links, 7 joints
Links:
- added link front_sensor; visual mesh filename=package://rubot_mecanum_description/meshes/nexus/urm04.STL scale=0.001 0.001 0.001
- added link left_sensor; visual mesh filename=package://rubot_mecanum_description/meshes/nexus/urm04.STL scale=0.001 0.001 0.001
- added link lower_left_wheel_shaft, mass 0.055; collision mesh filename=package://rubot_mecanum_description/meshes/nexus/wheel_shaf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 scale=0.001 0.001 0.001; visual mesh filename=package://rubot_mecanum_description/meshes/nexus/wheel_shaf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 scale=0.001 0.001 0.001
- added link lower_right_wheel_shaft, mass 0.055; collision mesh filename=package://rubot_mecanum_description/meshes/nexus/wheel_shaf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 scale=0.001 0.001 0.001; visual mesh filename=package://rubot_mecanum_description/meshes/nexus/wheel_shaf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 scale=0.001 0.001 0.001
- added link rear_sensor; visual mesh filename=package://rubot_mecanum_description/meshes/nexus/urm04.STL scale=0.001 0.001 0.001
- added link right_sensor; visual mesh filename=package://rubot_mecanum_description/meshes/nexus/urm04.STL scale=0.001 0.001 0.001
- added link upper_left_wheel_shaft, mass 0.055; collision mesh filename=package://rubot_mecanum_description/meshes/nexus/wheel_shaf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 scale=0.001 0.001 0.001; visual mesh filename=package://rubot_mecanum_description/meshes/nexus/wheel_shaf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 scale=0.001 0.001 0.001
- added link upper_right_wheel_shaft, mass 0.055; collision mesh filename=package://rubot_mecanum_description/meshes/nexus/wheel_shaf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 scale=0.001 0.001 0.001; visual mesh filename=package://rubot_mecanum_description/meshes/nexus/wheel_shaf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 scale=0.001 0.001 0.001
- link base_link: mass 10 -> 2.844; geometry collision mesh filename=package://rubot_mecanum_description/meshes/nexus/nexus_base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 scale=0.001 0.001 0.001; visual mesh filename=package://rubot_mecanum_description/meshes/nexus/nexus_base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 scale=0.001 0.001 0.001
- link camera: geometry collision box size=0.075 0.075 0.025; visual mesh filename=package://rubot_mecanum_description/meshes/nexus/piCamera.s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 scale=0.0025 0.0025 0.0025
- link lower_left_wheel: geometry collision cylinder length=0.0505 radius=0.05; visual mesh filename=package://rubot_mecanum_description/meshes/nexus/mecanum_wh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 scale=0.001 0.001 0.001
- link lower_right_wheel: geometry collision cylinder length=0.0505 radius=0.05; visual mesh filename=package://rubot_mecanum_description/meshes/nexus/mecanum_wh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 scale=0.001 0.001 0.001
- link upper_left_wheel: geometry collision cylinder length=0.0505 radius=0.05; visual mesh filename=package://rubot_mecanum_description/meshes/nexus/mecanum_wh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 scale=0.001 0.001 0.001
- link upper_right_wheel: geometry collision cylinder length=0.0505 radius=0.05; visual mesh filename=package://rubot_mecanum_description/meshes/nexus/mecanum_wh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 scale=0.001 0.001 0.001
Joints:
- added joint front_sensor_joint: type fixed, parent base_link, child front_sensor, origin xyz=0.205 0 0.010 rpy=0 0 0
- added joint left_sensor_joint: type fixed, parent base_link, child left_sensor, origin xyz=0 0.108 0.010 rpy=0 0 1.57079632679
- added joint lower_left_wheel_shaft_joint: type fixed, parent base_link, child lower_left_wheel_shaft, origin xyz=-0.150 0.108 0.0 rpy=0 0 0
- added joint lower_right_wheel_shaft_joint: type fixed, parent base_link, child lower_right_wheel_shaft, origin xyz=-0.150 -0.108 0.0 rpy=3.14159265359 0 0
- added joint rear_sensor_joint: type fixed, parent base_link, child rear_sensor, origin xyz=-0.201 0 0.010 rpy=0 0 3.14159265359
- added joint right_sensor_joint: type fixed, parent base_link, child right_sensor, origin xyz=0 -0.108 0.010 rpy=0 0 -1.57079632679
- added joint upper_left_wheel_shaft_joint: type fixed, parent base_link, child upper_left_wheel_shaft, origin xyz=0.150 0.108 0.0 rpy=0 0 0
- added joint upper_right_wheel_shaft_joint: type fixed, parent base_link, child upper_right_wheel_shaft, origin xyz=0.150 -0.108 0.0 rpy=3.14159265359 0 0
- joint base_link_joint: origin xyz=0 0 0 rpy=0 0 0 -> xyz=0 0 0.05 rpy=0 0 0
- joint joint_camera: axis 0 1 0 -> 0 0 1; origin xyz=0.236 0.076 0.072 rpy=0 0 0 -> xyz=0.2 0 0.05 rpy=0 0 0
- joint lower_left_wheel_joint: origin xyz=0 0 0 rpy=0 0 0 -> xyz=0 0.042 0 rpy=0 0 0; parent base_link -> lower_left_wheel_shaft
- joint lower_right_wheel_joint: origin xyz=0 0 0 rpy=0 0 0 -> xyz=0 0.042 0 rpy=0 0 0; parent base_link -> lower_right_wheel_shaft
- joint upper_left_wheel_joint: origin xyz=0 0 0 rpy=0 0 0 -> xyz=0 0.042 0 rpy=0 0 0; parent base_link -> upper_left_wheel_shaft
- joint upper_right_wheel_joint: origin xyz=0 0 0 rpy=0 0 0 -> xyz=0 0.042 0 rpy=0 0 0; parent base_link -> upper_right_wheel_shaft

Commit message: message

File: src/rubot_mecanum_description/urdf/rubot.urdf (robot description, URDF)
Before this commit: robot nexus, 16 links, 15 joints
Links:
- removed link front_sensor
- removed link left_sensor
- removed link lower_left_wheel_shaft
- removed link lower_right_wheel_shaft
- removed link rear_sensor
- removed link right_sensor
- removed link upper_left_wheel_shaft
- removed link upper_right_wheel_shaft
- link base_link: mass 2.844 -> 10; geometry collision box size=0.1 0.1 0.35; visual mesh filename=package://rubot_mecanum_description/meshes/rubot/base_link.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 scale=0.001 0.001 0.001
- link base_scan: geometry collision cylinder length=0.01575 radius=0.0275; visual mesh filename=package://rubot_mecanum_description/meshes/rubot/lidar.stl scale=0.001 0.001 0.001
- link camera: geometry collision box size=0.075 0.075 0.025; visual mesh filename=package://rubot_mecanum_description/meshes/rubot/picam.stl scale=0.001 0.001 0.001
- link lower_left_wheel: geometry collision mesh filename=package://rubot_mecanum_description/meshes/rubot/wheel_left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 scale=0.001 0.001 0.001; visual mesh filename=package://rubot_mecanum_description/meshes/rubot/wheel_left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 scale=0.001 0.001 0.001
- link lower_right_wheel: geometry collision mesh filename=package://rubot_mecanum_description/meshes/rubot/wheel_righ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 scale=0.001 0.001 0.001; visual mesh filename=package://rubot_mecanum_description/meshes/rubot/wheel_righ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 scale=0.001 0.001 0.001
- link upper_left_wheel: geometry collision mesh filename=package://rubot_mecanum_description/meshes/rubot/wheel_left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 scale=0.001 0.001 0.001; visual mesh filename=package://rubot_mecanum_description/meshes/rubot/wheel_left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 scale=0.001 0.001 0.001
- link upper_right_wheel: geometry collision mesh filename=package://rubot_mecanum_description/meshes/rubot/wheel_righ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 scale=0.001 0.001 0.001; visual mesh filename=package://rubot_mecanum_description/meshes/rubot/wheel_righ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 scale=0.001 0.001 0.001
Joints:
- removed joint front_sensor_joint
- removed joint left_sensor_joint
- removed joint lower_left_wheel_shaft_joint
- removed joint lower_right_wheel_shaft_joint
- removed joint rear_sensor_joint
- removed joint right_sensor_joint
- removed joint upper_left_wheel_shaft_joint
- removed joint upper_right_wheel_shaft_joint
- joint base_link_joint: origin xyz=0 0 0.05 rpy=0 0 0 -> xyz=0 0 0 rpy=0 0 0
- joint joint_camera: axis 0 0 1 -> 0 1 0; origin xyz=0.2 0 0.05 rpy=0 0 0 -> xyz=0.236 0.076 0.072 rpy=0 0 0
- joint lower_left_wheel_joint: origin xyz=0 0.042 0 rpy=0 0 0 -> xyz=0 0 0 rpy=0 0 0; parent lower_left_wheel_shaft -> base_link
- joint lower_right_wheel_joint: origin xyz=0 0.042 0 rpy=0 0 0 -> xyz=0 0 0 rpy=0 0 0; parent lower_right_wheel_shaft -> base_link
- joint scan_joint: origin xyz=0 0 0.09 rpy=0 0 3.14 -> xyz=0.111 0.076 0.124 rpy=0 0 3.14
- joint upper_left_wheel_joint: origin xyz=0 0.042 0 rpy=0 0 0 -> xyz=0 0 0 rpy=0 0 0; parent upper_left_wheel_shaft -> base_link
- joint upper_right_wheel_joint: origin xyz=0 0.042 0 rpy=0 0 0 -> xyz=0 0 0 rpy=0 0 0; parent upper_right_wheel_shaft -> base_link
